File: schematic/TACOS-ESP-Integrated-Full/TACOS-ESP-Integrated-Full.kicad_pcb (KiCad board)
At the start: 2 copper layers, 27 parts, among them J1 Relay, J2 MRC522, J3 Relay, J4 Vin, Q1 PN2222A, Q2 PN2222A, Q3 PN2222A, Q4 PN2222A, Q5 PN2222A, SW1 SW_ARM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

Commit message: schematic: update
Parts:
- D1: value ONLINE LED -> SYSTEM LED
- moved J2 21.5 mm to (41.2, 64.9), turned to 90 degrees
- moved J4 4.07 mm to (29.2, 31.8), turned to 270 degrees
- moved R12 1.53 mm to (63.5, 73.4)
- moved R3 0.93 mm to (50.0, 73.4)
- moved R8 0.46 mm to (44.9, 52.2)
Connections:
- R1 pad 1: GND -> SWITCH
- R1 pad 2: SWITCH -> GND
- R2 pad 1: GND -> Net-(D1-Pad1)
- R2 pad 2: Net-(D1-Pad1) -> GND
Routing:
- net 5V: track 170.4 -> 0.00 mm
- net GND: track 159.4 -> 0.00 mm
- net 3V3: track 84.1 -> 0.00 mm
- net ERROR_NET: track 73.4 -> 0.16 mm
- net Net-(D4-Pad1): track 51.9 -> 0.00 mm
- net POWER_NET: track 40.8 -> 0.00 mm, vias 1 -> 0
- net RST: track 35.2 -> 0.00 mm
- net STATUS_NET: track 33.6 -> 0.00 mm
- net MISO: track 26.8 -> 0.00 mm
- net Net-(J1-Pad1): track 25.7 -> 0.00 mm
- net SCK: track 24.8 -> 0.00 mm
- net Net-(D2-Pad1): track 26.2 -> 1.93 mm
- net SWITCH: track 21.5 -> 0.00 mm
- net MOSI: track 21.3 -> 0.00 mm
- net Net-(J3-Pad1): track 18.6 -> 0.00 mm
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
Commit message: schematic: update
Parts:
- added D5: D, Diode_SMD:D_0603_1608Metric, F.Cu at (79.4, 120.2)
- added D6: D, Diode_SMD:D_0603_1608Metric, F.Cu at (43.3, 83.7)
- added R13: R330, Resistor_SMD:R_0603_1608Metric, F.Cu at (38.3, 120.0)
- added R14: R1K, Resistor_SMD:R_0603_1608Metric, F.Cu at (50.3, 73.4)
- added R15: R1K, Resistor_SMD:R_0603_1608Metric, F.Cu at (112.6, 47.3)
- D2: value POWER LED -> Error LED
- D3: value POWER LED -> Power LED
- D4: value POWER LED -> Status LED
- J1: value Relay -> Power Relay
- J3: value Relay -> Error Relay
- R10, R11: value R? -> R4.7K; footprint Resistor_THT:R_Bare_Metal_Element_L12.4mm_W4.8mm_P11.40mm -> Resistor_SMD:R_0603_1608Metric
- moved D4 59.7 mm to (30.9, 120.4)
- moved Q4 51.9 mm to (76.4, 127.4), turned to 90 degrees
- moved R12 51.0 mm to (42.5, 119.9), turned to 90 degrees
- moved Q5 49.6 mm to (39.9, 124.1), turned to 270 degrees
- moved J3 39.7 mm to (85.8, 126.3)
- moved R11 38.0 mm to (74.4, 120.2), turned to 90 degrees
- moved R3 27.7 mm to (39.5, 99.0)
- moved R2 7.05 mm to (35.6, 48.4), turned to 90 degrees
Connections:
- D2 pad 2: 5V -> Net-(D2-Pad2)
- D3 pad 2: 5V -> Net-(D3-Pad2)
- D4 pad 2: 5V -> Net-(D4-Pad2)
- Q1 pad 1: Net-(Q1-Pad1) -> GND
- Q1 pad 2: POWER_NET -> Net-(Q1-Pad2)
- Q2 pad 1: Net-(Q2-Pad1) -> GND
- Q2 pad 2: POWER_NET -> Net-(Q2-Pad2)
- Q3 pad 1: Net-(Q3-Pad1) -> GND
- Q3 pad 2: ERROR_NET -> Net-(Q3-Pad2)
- Q4 pad 1: Net-(Q4-Pad1) -> GND
- Q4 pad 2: ERROR_NET -> Net-(Q4-Pad2)
- Q5 pad 1: Net-(Q5-Pad1) -> GND
- Q5 pad 2: STATUS_NET -> Net-(Q5-Pad2)
- R10 pad 1: Net-(Q2-Pad1) -> Net-(Q2-Pad2)
- R10 pad 2: GND -> POWER_NET
- R11 pad 1: Net-(Q4-Pad1) -> Net-(Q4-Pad2)
- R11 pad 2: GND -> ERROR_NET
- R12 pad 1: Net-(Q5-Pad1) -> Net-(Q5-Pad2)
- R12 pad 2: GND -> STATUS_NET
- R3 pad 1: Net-(Q3-Pad1) -> 5V
- R3 pad 2: GND -> Net-(D2-Pad2)
- R4 pad 1: Net-(Q1-Pad1) -> 5V
- R4 pad 2: GND -> Net-(D3-Pad2)

Commit message: schematic: update
Parts:
- removed J3: Error Relay, TerminalBlock:TerminalBlock_bornier-2_P5.08mm
- removed R1: R330, Resistor_SMD:R_0603_1608Metric
- added LS1: Error Speaker, TerminalBlock:TerminalBlock_bornier-2_P5.08mm, F.Cu at (73.6, 92.1)
- added SW2: SW_DEVICE_RST, TerminalBlock:TerminalBlock_bornier-2_P5.08mm, F.Cu at (29.4, 52.9)
- R11: value R4.7K -> R1K
- moved R15 75.8 mm to (40.1, 69.2)
- moved Q4 39.3 mm to (59.6, 91.9), turned to 0 degrees
- moved Q5 37.8 mm to (38.5, 86.3), turned to 180 degrees
- moved R11 37.5 mm to (58.9, 86.0)
- moved R3 37.3 mm to (67.4, 74.2), turned to 270 degrees
- moved D4 33.4 mm to (29.4, 87.0)
- moved D5 33.1 mm to (65.6, 90.0)
- moved R12 27.3 mm to (40.0, 92.8), turned to 0 degrees
- moved R13 27.2 mm to (36.2, 92.8), turned to 180 degrees
- moved R5 20.8 mm to (45.9, 60.3), turned to 270 degrees
- moved Q1 17.4 mm to (39.2, 62.8), turned to 180 degrees
- moved R6 16.8 mm to (48.4, 60.3), turned to 270 degrees
- moved R9 16.5 mm to (61.1, 60.3), turned to 270 degrees
- moved R7 13.7 mm to (51.0, 60.3), turned to 270 degrees
- moved R8 11.7 mm to (53.4, 60.3), turned to 270 degrees
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Connections:
- net 5V renamed +5V
- J2 pad 8: 3V3 -> (no net)
- SW1 pad 1: SWITCH -> GND
- SW1 pad 2: 3V3 -> SWITCH
- U1 pad 1: (no net) -> DEV_RST
- U1 pad 8: 3V3 -> (no net)
Routing:
- net +5V: track 0.39 -> 15.7 mm
- net Net-(D6-Pad2): track 0.00 -> 11.7 mm
- net Net-(D5-Pad2): track 0.00 -> 8.51 mm
- net Net-(D2-Pad1): track 1.93 -> 0.00 mm

Commit message: schematic: update - routed
Parts:
- added H1: MountingHole, MountingHole:MountingHole_2.7mm_M2.5_Pad, F.Cu at (31.8, 30.7)
- added H2: MountingHole, MountingHole:MountingHole_2.7mm_M2.5_Pad, F.Cu at (28.4, 69.1)
- added H3: MountingHole, MountingHole:MountingHole_2.7mm_M2.5_Pad, F.Cu at (90.1, 59.8)
- added H4: MountingHole, MountingHole:MountingHole_2.7mm_M2.5_Pad, F.Cu at (67.3, 30.6)
- moved LS1 62.7 mm to (90.4, 31.7), turned to 180 degrees
- moved R13 58.3 mm to (89.7, 69.7), turned to 0 degrees
- moved D4 57.0 mm to (85.3, 75.9), turned to 0 degrees
- moved R12 56.1 mm to (89.8, 66.8)
- moved Q4 55.4 mm to (90.2, 45.7), turned to 90 degrees
- moved D5 55.2 mm to (88.3, 39.7), turned to 0 degrees
- moved Q5 50.6 mm to (84.6, 65.6), turned to 270 degrees
- moved R11 49.2 mm to (85.3, 44.4), turned to 180 degrees
- moved D2 48.7 mm to (78.5, 31.7), turned to 180 degrees
- moved J4 45.2 mm to (29.0, 75.9), turned to 0 degrees
- moved J1 44.3 mm to (73.7, 75.9), turned to 0 degrees
- moved D6 42.1 mm to (76.7, 69.8), turned to 180 degrees
- moved R10 40.2 mm to (79.6, 66.1), turned to 180 degrees
- moved Q3 39.3 mm to (78.4, 45.6), turned to 90 degrees
- moved R3 37.2 mm to (74.2, 37.6), turned to 180 degrees
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Routing:
- net +5V: track 15.7 -> 198.0 mm
- net POWER_NET: track 0.00 -> 86.8 mm
- net STATUS_NET: track 0.00 -> 84.3 mm
- net ERROR_NET: track 0.00 -> 78.4 mm
- net SWITCH: track 0.00 -> 34.8 mm
- net SS: track 0.00 -> 28.4 mm
- net DEV_RST: track 0.00 -> 25.1 mm
- net RST: track 0.00 -> 21.0 mm
- net MOSI: track 0.00 -> 16.3 mm
- net SCK: track 0.00 -> 12.0 mm
- net Net-(D2-Pad1): track 0.00 -> 11.3 mm
- net MISO: track 0.00 -> 8.67 mm
- net Net-(D4-Pad1): track 0.00 -> 8.15 mm
- net Net-(Q2-Pad2): track 0.00 -> 7.40 mm
- net Net-(D3-Pad1): track 0.00 -> 7.24 mm
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- added copper zone on B.Cu, net GND
- added copper zone on F.Cu, net GND
Other:
- board outline added: 69.6 x 57.9 mm
- net class Default: trace_width 0.25 -> 0.5
- rule trace_min: 0.2 -> 0.5
- board text added: "TACOS-ESP-Integrated v1"
- board text added: "https://github.com/vhs/tacos-esp-integrated"

Commit message: schematic: updates
Parts:
- H1, H2, H3, H4: footprint MountingHole:MountingHole_2.7mm_M2.5_Pad -> MountingHole:MountingHole_3.2mm_M3_Pad
- moved J2 42.9 mm to (20.5, 60.8)
- moved R6 33.4 mm to (25.2, 56.5), turned to 180 degrees
- moved R5 33.4 mm to (25.2, 60.0), turned to 180 degrees
- moved R7 33.3 mm to (25.2, 53.2), turned to 180 degrees
- moved R8 33.3 mm to (25.2, 49.2), turned to 180 degrees
- moved R9 33.3 mm to (25.2, 44.8), turned to 180 degrees
- moved U1 33.0 mm to (32.0, 26.0), turned to 0 degrees
- moved H4 29.0 mm to (96.2, 29.0)
- moved H3 19.3 mm to (96.5, 78.0)
- moved H2 11.1 mm to (21.8, 78.0)
- moved H1 10.5 mm to (21.5, 28.8)
- moved SW1 4.49 mm to (65.8, 31.5)
- moved D2 0.79 mm to (77.7, 31.5)
- moved D5 0.79 mm to (87.6, 39.5)
- moved LS1 0.79 mm to (89.7, 31.5)
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Connections:
- J2 pad 8: (no net) -> +3V3
- U1 pad 8: (no net) -> +3V3
Routing:
- net +5V: track 198.0 -> 150.0 mm
- net ERROR_NET: track 78.4 -> 34.2 mm, vias 0 -> 1
- net STATUS_NET: track 84.3 -> 47.2 mm, vias 0 -> 1
- net POWER_NET: track 86.8 -> 49.7 mm
- net DEV_RST: track 25.1 -> 59.8 mm
- net SWITCH: track 34.8 -> 5.98 mm
- net SCK: track 12.0 -> 25.3 mm
- net +3V3: track 0.00 -> 11.8 mm
- net SS: track 28.4 -> 21.2 mm
- net MISO: track 8.67 -> 15.6 mm, vias 0 -> 1
- net RST: track 21.0 -> 16.1 mm
- net Net-(D6-Pad2): track 10.8 -> 15.6 mm
- net MOSI: track 16.3 -> 18.6 mm, vias 0 -> 1
- net Net-(J2-Pad3): track 6.13 -> 4.96 mm
- net GND: vias 0 -> 1
Other:
- board size 69.6 x 57.9 mm -> 83.5 x 58 mm

Commit message: schematic: updates
Parts:
- added G***: LOGO, TACOS-ESP-Integrated:VHS logo - 150dpi, F.Cu at (73.0, 55.0)
- added SW3: SW_DEV_RST, Button_Switch_SMD:SW_SPST_PTS645, F.Cu at (43.8, 60.2)
- SW2: value SW_DEVICE_RST -> SW_DEV_RST
- moved R5 22.3 mm to (26.5, 37.8)
- moved J4 12.8 mm to (23.2, 64.2), turned to 270 degrees
- moved J2 3.76 mm to (20.2, 57.0)
- moved R10 3.49 mm to (75.8, 65.0), turned to 90 degrees
- moved R9 3.25 mm to (26.5, 41.8)
- moved R15 3.02 mm to (64.8, 65.0), turned to 90 degrees
- moved Q1 2.76 mm to (59.6, 64.5)
- moved Q5 2.49 mm to (81.9, 64.5)
- moved R6 2.36 mm to (26.5, 54.5)
- moved Q2 2.26 mm to (71.0, 64.5)
- moved D1 2.25 mm to (37.4, 75.9)
- moved D3 2.25 mm to (59.6, 75.9)
- moved D4 2.25 mm to (82.6, 75.9)
- moved D6 2.25 mm to (74.0, 69.8)
- moved J1 2.25 mm to (71.0, 75.9)
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Routing:
- net Net-(J2-Pad1): track 4.27 -> 26.1 mm
- net +5V: track 150.0 -> 167.0 mm
- net SS: track 21.2 -> 6.32 mm, vias 0 -> 1
- net DEV_RST: track 59.8 -> 63.5 mm
- net RST: track 16.1 -> 12.6 mm
- net MOSI: track 18.6 -> 15.3 mm, vias 1 -> 0
- net Net-(D5-Pad2): track 12.4 -> 15.4 mm
- net Net-(D6-Pad2): track 15.6 -> 12.8 mm
- net POWER_NET: track 49.7 -> 47.1 mm
- net Net-(Q2-Pad2): track 7.40 -> 4.76 mm
- net STATUS_NET: track 47.2 -> 44.6 mm, vias 1 -> 0
- net +3V3: track 11.8 -> 13.6 mm
- net Net-(D3-Pad1): track 7.24 -> 8.83 mm
- net SCK: track 25.3 -> 24.0 mm
- net Net-(J2-Pad7): track 4.28 -> 5.47 mm
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Other:
- board text added: "+"
- board text added: "-"
- board text added: "3V3"
- board text added: "GND"
- board text added: "IRQ"
- board text added: "MISO"
- board text added: "MOSI"
- board text added: "RST"
- board text added: "Rev: 2022-02-12"
- board text added: "SCK"
- board text added: "SS"

Commit message: schematic: updates
Parts:
- removed G***: LOGO, TACOS-ESP-Integrated:VHS logo - 150dpi
- added C1: CP, Capacitor_THT:CP_Radial_D5.0mm_P2.50mm, F.Cu at (32.0, 68.0)
- moved SW3 1.06 mm to (44.5, 61.0)
Other:
- board text added: "TACOS-ESP-Integrated v0.0.1"
- board text removed: "TACOS-ESP-Integrated v1"

Commit message: schematic: updates - redid routing - redid logo
Parts:
- added G***: LOGO, TACOS-ESP-Integrated:VHS logo - 150dpi, F.Cu at (74.5, 54.5)
Routing:
- net SS: track 6.32 -> 23.5 mm, vias 1 -> 0
- net +5V: track 167.4 -> 152.6 mm
- net STATUS_NET: track 44.6 -> 49.9 mm
- net Net-(D6-Pad2): track 12.8 -> 15.9 mm
- net Net-(D5-Pad2): track 15.4 -> 12.4 mm
- net MOSI: track 15.3 -> 16.5 mm, vias 0 -> 1
- net SCK: track 24.0 -> 22.8 mm
- net POWER_NET: track 47.1 -> 47.7 mm
- net ERROR_NET: track 34.0 -> 34.2 mm, vias 0 -> 1
- net MISO: vias 0 -> 1
Other:
- board text added: "TACOS-ESP-Integrated v0.0.2"
- board text removed: "TACOS-ESP-Integrated v0.0.1"
